File: pcb/SNES_MR_DeJitter_QID.brd (EAGLE design)
At the start: 85.2 x 26.4 mm, 92 parts, among them J1 SNESCART_CONN_SPARSE_4, U1 SuperCIC_lock, U2 uIGR, U3 EPM7032AETC44-10N, U4 74HCT2G125DP, U5 CDCE913, U6 2G17TI_DBV, U7 TLV70033, U8 TLV70018, U9 TSH122ICT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

Commit message: resolve inconsistency between schematic and BOM
Parts:
- R92: value 2k -> 6k19
- R93: value 623 -> 523
Changed lines of the file:
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@@
 <?xml version="1.0" encoding="utf-8"?>
 <!DOCTYPE eagle SYSTEM "eagle.dtd">
-<eagle version="9.5.2">
+<eagle version="9.6.2">
 <drawing>
 <settings>
@@
 <attribute name="VALUE" x="55.372" y="1.524" size="0.0254" layer="27"/>
 </element>
-<element name="R92" library="rcl" package="R0603" value="2k" x="58.674" y="21.336" smashed="yes">
+<element name="R92" library="rcl" package="R0603" value="6k19" x="58.674" y="21.336" smashed="yes">
 <attribute name="NAME" x="57.15" y="21.59" size="0.8128" layer="25" font="vector" ratio="15" rot="R180"/>
 </element>
@@
 <attribute name="NAME" x="60.579" y="18.415" size="0.8128" layer="25" font="vector" ratio="15"/>
 </element>
-<element name="R93" library="rcl" package="R0603" value="623" x="56.896" y="19.304" smashed="yes" rot="R180">
+<element name="R93" library="rcl" package="R0603" value="523" x="56.896" y="19.304" smashed="yes" rot="R180">
 <attribute name="NAME" x="56.896" y="18.542" size="0.8128" layer="25" font="vector" ratio="15" rot="R270"/>
 </element>
